Commit message: add lidar simulation

File: src/robot_pkg/description/robot.urdf.xacro (robot description, xacro)
@@ -3,3 +3,4 @@
     <xacro:include filename="robot_core.xacro"/>
     <xacro:include filename="gazebo_control.xacro"/>
+    <xacro:include filename="lidar.xacro"/>
 </robot>

File: src/robot_pkg/description/robot_core.xacro (robot description, xacro)
@@ -202,28 +202,3 @@
         <mu2 value="0.001"/>
     </gazebo>
-    <!-- LIDAR -->
-    <joint name="lidar_joint" type="fixed">
-        <parent link="base_link"/>
-        <child link="lidar"/>
-        <origin xyz="0 0 ${(0.058/2)+0.056+0.040}" rpy="0 0 0"/>
-    </joint>
-    <link name="lidar">
-        <visual>
-            <geometry>
-                <cylinder radius="0.033" length="0.058"/>
-            </geometry>
-            <material name="blue"/>
-        </visual>
-        <collision>
-            <geometry>
-                <cylinder radius="0.033" length="0.058"/>
-            </geometry>
-        </collision>
-    </link>
-    <joint name="laser_joint" type="fixed">
-        <parent link="base_link"/>
-        <child link="laser"/>
-        <origin xyz="0 0 ${0.042+0.056+0.040}" rpy="0 0 0"/>
-    </joint>
-    <link name="laser"/>
 </robot>

Commit message: add simulated ros2 control

File: src/robot_pkg/description/robot.urdf.xacro (robot description, xacro)
@@ -1,6 +1,13 @@
 <?xml version="1.0"?>
-<robot xmlns:xacro="http://www.ros.org/wiki/xacro" name="robot">
-    <xacro:include filename="robot_core.xacro"/>
-    <xacro:include filename="gazebo_control.xacro"/>
-    <xacro:include filename="lidar.xacro"/>
+<robot xmlns:xacro="http://www.ros.org/wiki/xacro"  name="robot">
+    <xacro:arg name="use_ros2_control" default="true"/>
+    <xacro:arg name="sim_mode" default="false"/>
+    <xacro:include filename="robot_core.xacro" />
+    <xacro:if value="$(arg use_ros2_control)">
+        <xacro:include filename="ros2_control.xacro" />
+    </xacro:if>
+    <xacro:unless value="$(arg use_ros2_control)">
+        <xacro:include filename="gazebo_control.xacro" />
+    </xacro:unless>
+    <xacro:include filename="lidar.xacro" />
 </robot>

File: src/robot_pkg/description/robot_core.xacro (robot description, xacro)
@@ -1,4 +1,14 @@
 <?xml version="1.0"?>
 <robot xmlns:xacro="http://www.ros.org/wiki/xacro">
+    <xacro:property name="motor_wheel_diameter" value="0.050"/>
+    <xacro:property name="motor_wheel_width" value="0.020"/>
+    <xacro:property name="motor_wheel_separation" value="0.114"/> <!--center to center-->
+    <xacro:property name="encoder_wheel_diameter" value="0.050"/>
+    <xacro:property name="encoder_wheel_width" value="0.005"/>
+    <xacro:property name="encoder_wheel_separation" value="0.142"/> <!--center to center-->
+    <xacro:property name="chassis_base_height" value="0.065"/>
+    <xacro:property name="chassis_width" value="0.200"/>
+    <xacro:property name="chassis_length" value="0.200"/>
+    <xacro:property name="chassis_height" value="0.056"/>
     <material name="blue">
         <color rgba="0.2 0.2 1 1"/>
@@ -13,6 +23,5 @@
         <color rgba="0.5 0.2 0 1"/>
     </material>
-    <link name="base_link">
-    </link>
+    <link name="base_link"></link>
     <joint name="synthetic_mass_joint" type="fixed">
         <parent link="base_link"/>
@@ -31,10 +40,10 @@
         <parent link="base_link"/>
         <child link="chassis"/>
-        <origin xyz="0 0 ${(65-25+56/2)*1e-3}"/> <!-- 65mm - 50mm/2 : height of the chassis above the motors axles -->
+        <origin xyz="0 0 ${chassis_base_height - motor_wheel_diameter/2 + chassis_height/2}"/>
     </joint>
     <link name="chassis">
         <visual>
             <geometry>
-                <box size="0.200 0.200 0.056"/>
+                <box size="${chassis_length} ${chassis_width} ${chassis_height}"/>
                 <material name="brown"/>
             </geometry>
@@ -42,6 +51,5 @@
         <collision>
             <geometry>
-                <box size="0.200 0.200 0.056"/>
-                <material name="brown"/>
+                <box size="${chassis_length} ${chassis_width} ${chassis_height}"/>
             </geometry>
         </collision>
@@ -51,5 +59,5 @@
         <parent link="base_link"/>
         <child link="motor_left_wheel"/>
-        <origin xyz="0 0.047 0" rpy="-${pi/2} 0 0"/>
+        <origin xyz="0 ${motor_wheel_separation/2} 0" rpy="-${pi/2} 0 0"/>
         <axis xyz="0 0 1"/>
     </joint>
@@ -57,5 +65,5 @@
         <visual>
             <geometry>
-                <cylinder radius="0.025" length="0.020"/>
+                <cylinder radius="${motor_wheel_diameter/2}" length="${motor_wheel_width/2}"/>
             </geometry>
             <material name="white"/>
@@ -63,5 +71,5 @@
         <collision>
             <geometry>
-                <cylinder radius="0.025" length="0.020"/>
+                <cylinder radius="${motor_wheel_diameter/2}" length="${motor_wheel_width/2}"/>
             </geometry>
         </collision>
@@ -75,5 +83,5 @@
         <parent link="base_link"/>
         <child link="motor_right_wheel"/>
-        <origin xyz="0 -0.047 0" rpy="${pi/2} 0 0"/>
+        <origin xyz="0 -${motor_wheel_separation/2} 0" rpy="${pi/2} 0 0"/>
         <axis xyz="0 0 -1"/>
     </joint>
@@ -81,5 +89,5 @@
         <visual>
             <geometry>
-                <cylinder radius="0.025" length="0.020"/>
+                <cylinder radius="${motor_wheel_diameter/2}" length="${motor_wheel_width/2}"/>
             </geometry>
             <material name="white"/>
@@ -87,5 +95,5 @@
         <collision>
             <geometry>
-                <cylinder radius="0.025" length="0.020"/>
+                <cylinder radius="${motor_wheel_diameter/2}" length="${motor_wheel_width/2}"/>
             </geometry>
         </collision>
@@ -100,5 +108,5 @@
         <parent link="base_link"/>
         <child link="encoder_left_wheel"/>
-        <origin xyz="0 0.071 0" rpy="-${pi/2} 0 0"/>
+        <origin xyz="0 ${encoder_wheel_separation/2} 0" rpy="-${pi/2} 0 0"/>
         <axis xyz="0 0 1"/>
     </joint>
@@ -106,28 +114,17 @@
         <visual>
             <geometry>
-                <cylinder radius="0.025" length="0.0025"/>
+                <cylinder radius="${encoder_wheel_diameter/2}" length="${encoder_wheel_width/2}"/>
             </geometry>
             <material name="grey"/>
         </visual>
-        <collision>
-            <geometry>
-                <cylinder radius="0.020" length="0.0025"/>
-            </geometry>
-        </collision>
         <inertial>
             <mass value="0.01"/>
-            <origin xyz="0.0 0.0 0.025" rpy="0.0 0.0 0.0"/>
             <inertia ixx="0.000007" ixy="0.0" ixz="0.0" iyy="0.000007" iyz="0.0" izz="0.000008"/>
         </inertial>
     </link>
-    <gazebo reference="encoder_left_wheel">
-        <material>Gazebo/White</material>
-        <mu1 value="0.001"/>
-        <mu2 value="0.001"/>
-    </gazebo>
     <joint name="encoder_right_wheel_joint" type="continuous">
         <parent link="base_link"/>
         <child link="encoder_right_wheel"/>
-        <origin xyz="0 -0.071 0" rpy="${pi/2} 0 0"/>
+        <origin xyz="0 -${encoder_wheel_separation/2} 0" rpy="${pi/2} 0 0"/>
         <axis xyz="0 0 -1"/>
     </joint>
@@ -135,34 +132,23 @@
         <visual>
             <geometry>
-                <cylinder radius="0.025" length="0.0025"/>
+                <cylinder radius="${encoder_wheel_diameter/2}" length="${encoder_wheel_width/2}"/>
             </geometry>
             <material name="grey"/>
         </visual>
-        <collision>
-            <geometry>
-                <cylinder radius="0.020" length="0.0025"/>
-            </geometry>
-        </collision>
         <inertial>
             <mass value="0.01"/>
-            <origin xyz="0.0 0.0 0.025" rpy="0.0 0.0 0.0"/>
             <inertia ixx="0.000007" ixy="0.0" ixz="0.0" iyy="0.000007" iyz="0.0" izz="0.000008"/>
         </inertial>
     </link>
-    <gazebo reference="encoder_right_wheel">
-        <material>Gazebo/White</material>
-        <mu1 value="0.001"/>
-        <mu2 value="0.001"/>
-    </gazebo>
     <!-- CASTER WHEELS -->
     <joint name="front_caster_wheel_joint" type="fixed">
         <parent link="base_link"/>
         <child link="front_caster_wheel"/>
-        <origin xyz="0.080 0 0.0075" rpy="${pi} 0 0"/>
+        <origin xyz="0.080 0 0" rpy="${pi} 0 0"/>
     </joint>
     <link name="front_caster_wheel">
         <visual>
             <geometry>
-                <cylinder radius="0.01" length="0.065"/>
+                <cylinder radius="0.01" length="${chassis_base_height}"/>
             </geometry>
             <material name="white"/>
@@ -170,5 +156,5 @@
         <collision>
             <geometry>
-                <cylinder radius="0.01" length="0.063"/>
+                <cylinder radius="0.01" length="${chassis_base_height-2}"/>
             </geometry>
         </collision>
@@ -182,10 +168,10 @@
         <parent link="base_link"/>
         <child link="back_caster_wheel"/>
-        <origin xyz="-0.080 0 0.0075" rpy="0 0 0"/>
+        <origin xyz="-0.080 0 0" rpy="0 0 0"/>
     </joint>
     <link name="back_caster_wheel">
         <visual>
             <geometry>
-                <cylinder radius="0.01" length="0.065"/>
+                <cylinder radius="0.01" length="${chassis_base_height}"/>
             </geometry>
             <material name="white"/>
@@ -193,5 +179,5 @@
         <collision>
             <geometry>
-                <cylinder radius="0.01" length="0.063"/>
+                <cylinder radius="0.01" length="${chassis_base_height-2}"/>
             </geometry>
         </collision>
