Commit message: basic simulation of the robot

File: src/robot_pkg/description/robot_core.xacro (robot description, xacro)
@@ -14,4 +14,11 @@
     </material>
     <link name="base_link">
+    </link>
+    <joint name="synthetic_mass_joint" type="fixed">
+        <parent link="base_link"/>
+        <child link="synthetic_mass"/>
+        <origin xyz="0 0 0" rpy="0 0 0"/>
+    </joint>
+    <link name="synthetic_mass">
         <inertial>
             <mass value="1.0"/>
@@ -41,5 +48,5 @@
     </link>
     <!-- MOTOR WHEELS -->
-    <joint name="motor_left_wheel_joint" type="continuous">
+    <joint name="left_wheel_joint" type="continuous">
         <parent link="base_link"/>
         <child link="motor_left_wheel"/>
@@ -59,6 +66,11 @@
             </geometry>
         </collision>
-    </link>
-    <joint name="motor_right_wheel_joint" type="continuous">
+        <inertial>
+            <mass value="0.1"/>
+            <origin xyz="0.0 0.0 0.025" rpy="0.0 0.0 0.0"/>
+            <inertia ixx="0.00007" ixy="0.0" ixz="0.0" iyy="0.00007" iyz="0.0" izz="0.00008"/>
+        </inertial>
+    </link>
+    <joint name="right_wheel_joint" type="continuous">
         <parent link="base_link"/>
         <child link="motor_right_wheel"/>
@@ -78,4 +90,9 @@
             </geometry>
         </collision>
+        <inertial>
+            <mass value="0.1"/>
+            <origin xyz="0.0 0.0 0.025" rpy="0.0 0.0 0.0"/>
+            <inertia ixx="0.00007" ixy="0.0" ixz="0.0" iyy="0.00007" iyz="0.0" izz="0.00008"/>
+        </inertial>
     </link>
      <!-- ENCODER WHEELS -->
@@ -95,8 +112,18 @@
         <collision>
             <geometry>
-                <cylinder radius="0.025" length="0.0025"/>
-            </geometry>
-        </collision>
-    </link>
+                <cylinder radius="0.020" length="0.0025"/>
+            </geometry>
+        </collision>
+        <inertial>
+            <mass value="0.01"/>
+            <origin xyz="0.0 0.0 0.025" rpy="0.0 0.0 0.0"/>
+            <inertia ixx="0.000007" ixy="0.0" ixz="0.0" iyy="0.000007" iyz="0.0" izz="0.000008"/>
+        </inertial>
+    </link>
+    <gazebo reference="encoder_left_wheel">
+        <material>Gazebo/White</material>
+        <mu1 value="0.001"/>
+        <mu2 value="0.001"/>
+    </gazebo>
     <joint name="encoder_right_wheel_joint" type="continuous">
         <parent link="base_link"/>
@@ -114,8 +141,18 @@
         <collision>
             <geometry>
-                <cylinder radius="0.025" length="0.0025"/>
-            </geometry>
-        </collision>
-    </link>
+                <cylinder radius="0.020" length="0.0025"/>
+            </geometry>
+        </collision>
+        <inertial>
+            <mass value="0.01"/>
+            <origin xyz="0.0 0.0 0.025" rpy="0.0 0.0 0.0"/>
+            <inertia ixx="0.000007" ixy="0.0" ixz="0.0" iyy="0.000007" iyz="0.0" izz="0.000008"/>
+        </inertial>
+    </link>
+    <gazebo reference="encoder_right_wheel">
+        <material>Gazebo/White</material>
+        <mu1 value="0.001"/>
+        <mu2 value="0.001"/>
+    </gazebo>
     <!-- CASTER WHEELS -->
     <joint name="front_caster_wheel_joint" type="fixed">
@@ -133,8 +170,13 @@
         <collision>
             <geometry>
-                <cylinder radius="0.01" length="0.065"/>
-            </geometry>
-        </collision>
-    </link>
+                <cylinder radius="0.01" length="0.063"/>
+            </geometry>
+        </collision>
+    </link>
+    <gazebo reference="front_caster_wheel">
+        <material>Gazebo/Grey</material>
+        <mu1 value="0.001"/>
+        <mu2 value="0.001"/>
+    </gazebo>
     <joint name="back_caster_wheel_joint" type="fixed">
         <parent link="base_link"/>
@@ -151,8 +193,13 @@
         <collision>
             <geometry>
-                <cylinder radius="0.01" length="0.065"/>
-            </geometry>
-        </collision>
-    </link>
+                <cylinder radius="0.01" length="0.063"/>
+            </geometry>
+        </collision>
+    </link>
+    <gazebo reference="back_caster_wheel">
+        <material>Gazebo/Grey</material>
+        <mu1 value="0.001"/>
+        <mu2 value="0.001"/>
+    </gazebo>
     <!-- LIDAR -->
     <joint name="lidar_joint" type="fixed">

Commit message: correct urdf for caster wheels hight offset

File: src/robot_pkg/description/robot_core.xacro (robot description, xacro)
@@ -145,5 +145,5 @@
         <parent link="base_link"/>
         <child link="front_caster_wheel"/>
-        <origin xyz="0.080 0 0" rpy="${pi} 0 0"/>
+        <origin xyz="0.080 0 ${chassis_base_height/2 - motor_wheel_diameter/2}" rpy="${pi} 0 0"/>
     </joint>
     <link name="front_caster_wheel">
@@ -168,5 +168,5 @@
         <parent link="base_link"/>
         <child link="back_caster_wheel"/>
-        <origin xyz="-0.080 0 0" rpy="0 0 0"/>
+        <origin xyz="-0.080 0 ${chassis_base_height/2 - motor_wheel_diameter/2}" rpy="0 0 0"/>
     </joint>
     <link name="back_caster_wheel">

Commit message: correct bugs

File: src/robot_pkg/description/robot_core.xacro (robot description, xacro)
@@ -65,5 +65,5 @@
         <visual>
             <geometry>
-                <cylinder radius="${motor_wheel_diameter/2}" length="${motor_wheel_width/2}"/>
+                <cylinder radius="${motor_wheel_diameter/2}" length="${motor_wheel_width}"/>
             </geometry>
             <material name="white"/>
@@ -71,10 +71,10 @@
         <collision>
             <geometry>
-                <cylinder radius="${motor_wheel_diameter/2}" length="${motor_wheel_width/2}"/>
+                <cylinder radius="${motor_wheel_diameter/2}" length="${motor_wheel_width}"/>
             </geometry>
         </collision>
         <inertial>
             <mass value="0.1"/>
-            <origin xyz="0.0 0.0 0.025" rpy="0.0 0.0 0.0"/>
+            <origin xyz="0.0 0.0 0.01" rpy="0.0 0.0 0.0"/>
             <inertia ixx="0.00007" ixy="0.0" ixz="0.0" iyy="0.00007" iyz="0.0" izz="0.00008"/>
         </inertial>
@@ -89,5 +89,5 @@
         <visual>
             <geometry>
-                <cylinder radius="${motor_wheel_diameter/2}" length="${motor_wheel_width/2}"/>
+                <cylinder radius="${motor_wheel_diameter/2}" length="${motor_wheel_width}"/>
             </geometry>
             <material name="white"/>
@@ -95,10 +95,10 @@
         <collision>
             <geometry>
-                <cylinder radius="${motor_wheel_diameter/2}" length="${motor_wheel_width/2}"/>
+                <cylinder radius="${motor_wheel_diameter/2}" length="${motor_wheel_width}"/>
             </geometry>
         </collision>
         <inertial>
             <mass value="0.1"/>
-            <origin xyz="0.0 0.0 0.025" rpy="0.0 0.0 0.0"/>
+            <origin xyz="0.0 0.0 0.01" rpy="0.0 0.0 0.0"/>
             <inertia ixx="0.00007" ixy="0.0" ixz="0.0" iyy="0.00007" iyz="0.0" izz="0.00008"/>
         </inertial>
@@ -120,4 +120,5 @@
         <inertial>
             <mass value="0.01"/>
+            <origin xyz="0.0 0.0 0.01" rpy="0.0 0.0 0.0"/>
             <inertia ixx="0.000007" ixy="0.0" ixz="0.0" iyy="0.000007" iyz="0.0" izz="0.000008"/>
         </inertial>
@@ -138,4 +139,5 @@
         <inertial>
             <mass value="0.01"/>
+            <origin xyz="0.0 0.0 0.01" rpy="0.0 0.0 0.0"/>
             <inertia ixx="0.000007" ixy="0.0" ixz="0.0" iyy="0.000007" iyz="0.0" izz="0.000008"/>
         </inertial>
@@ -156,5 +158,5 @@
         <collision>
             <geometry>
-                <cylinder radius="0.01" length="${chassis_base_height-2}"/>
+                <cylinder radius="0.01" length="${chassis_base_height-0.002}"/>
             </geometry>
         </collision>
@@ -179,5 +181,5 @@
         <collision>
             <geometry>
-                <cylinder radius="0.01" length="${chassis_base_height-2}"/>
+                <cylinder radius="0.01" length="${chassis_base_height-0.002}"/>
             </geometry>
         </collision>

File: src/robot_pkg/description/ros2_control.xacro (robot description, xacro)
@@ -52,4 +52,12 @@
                 <state_interface name="position"/>
             </joint>
+            <!-- <joint name="encoder_left_wheel_joint">
+                <state_interface name="velocity"/>
+                <state_interface name="position"/>
+            </joint>
+            <joint name="encoder_right_wheel_joint">
+                <state_interface name="velocity"/>
+                <state_interface name="position"/>
+            </joint> -->
         </ros2_control>
     </xacro:if>
