Commit message: commit because long time without doing it... dont bother with change track

File: src/robot_pkg/description/gazebo_control.xacro (robot description, xacro)
@@ -6,5 +6,5 @@
             <left_joint>left_wheel_joint</left_joint>
             <right_joint>right_wheel_joint</right_joint>
-            <wheel_separation>0.114</wheel_separation>
+            <wheel_separation>0.146</wheel_separation>
             <wheel_diameter>0.050</wheel_diameter>
             <!-- Limits -->

File: src/robot_pkg/description/lidar.xacro (robot description, xacro)
@@ -41,7 +41,13 @@
                 </scan>
                 <range>
-                    <min>0.12</min>
-                    <max>12</max>
+                    <min>0.2</min>
+                    <max>6</max>
                 </range>
+                <noise>
+                    <!-- Use gaussian noise -->
+                    <type>gaussian</type>
+                    <mean>0.0</mean>
+                    <stddev>0.005</stddev>
+                </noise>
             </ray>
             <plugin name="laser_controller" filename="libgazebo_ros_ray_sensor.so">

File: src/robot_pkg/description/robot.urdf.xacro (robot description, xacro)
@@ -11,3 +11,4 @@
     </xacro:unless>
     <xacro:include filename="lidar.xacro" />
+    <xacro:include filename="imu.xacro" />
 </robot>

File: src/robot_pkg/description/robot_core.xacro (robot description, xacro)
@@ -2,9 +2,6 @@
 <robot xmlns:xacro="http://www.ros.org/wiki/xacro">
     <xacro:property name="motor_wheel_diameter" value="0.050"/>
-    <xacro:property name="motor_wheel_width" value="0.020"/>
-    <xacro:property name="motor_wheel_separation" value="0.114"/> <!--center to center-->
-    <xacro:property name="encoder_wheel_diameter" value="0.050"/>
-    <xacro:property name="encoder_wheel_width" value="0.005"/>
-    <xacro:property name="encoder_wheel_separation" value="0.142"/> <!--center to center-->
+    <xacro:property name="motor_wheel_width" value="0.005"/>
+    <xacro:property name="motor_wheel_separation" value="0.146"/> <!--center to center-->
     <xacro:property name="chassis_base_height" value="0.065"/>
     <xacro:property name="chassis_width" value="0.200"/>
@@ -104,43 +101,4 @@
         </inertial>
     </link>
-     <!-- ENCODER WHEELS -->
-    <joint name="encoder_left_wheel_joint" type="continuous">
-        <parent link="base_link"/>
-        <child link="encoder_left_wheel"/>
-        <origin xyz="0 ${encoder_wheel_separation/2} 0" rpy="-${pi/2} 0 0"/>
-        <axis xyz="0 0 1"/>
-    </joint>
-    <link name="encoder_left_wheel">
-        <visual>
-            <geometry>
-                <cylinder radius="${encoder_wheel_diameter/2}" length="${encoder_wheel_width/2}"/>
-            </geometry>
-            <material name="grey"/>
-        </visual>
-        <inertial>
-            <mass value="0.01"/>
-            <origin xyz="0.0 0.0 0.01" rpy="0.0 0.0 0.0"/>
-            <inertia ixx="0.000007" ixy="0.0" ixz="0.0" iyy="0.000007" iyz="0.0" izz="0.000008"/>
-        </inertial>
-    </link>
-    <joint name="encoder_right_wheel_joint" type="continuous">
-        <parent link="base_link"/>
-        <child link="encoder_right_wheel"/>
-        <origin xyz="0 -${encoder_wheel_separation/2} 0" rpy="${pi/2} 0 0"/>
-        <axis xyz="0 0 -1"/>
-    </joint>
-    <link name="encoder_right_wheel">
-        <visual>
-            <geometry>
-                <cylinder radius="${encoder_wheel_diameter/2}" length="${encoder_wheel_width/2}"/>
-            </geometry>
-            <material name="grey"/>
-        </visual>
-        <inertial>
-            <mass value="0.01"/>
-            <origin xyz="0.0 0.0 0.01" rpy="0.0 0.0 0.0"/>
-            <inertia ixx="0.000007" ixy="0.0" ixz="0.0" iyy="0.000007" iyz="0.0" izz="0.000008"/>
-        </inertial>
-    </link>
     <!-- CASTER WHEELS -->
     <joint name="front_caster_wheel_joint" type="fixed">

File: src/robot_pkg/description/ros2_control.xacro (robot description, xacro)
@@ -61,12 +61,4 @@
                 <state_interface name="position"/>
             </joint>
-            <!-- <joint name="encoder_left_wheel_joint">
-                <state_interface name="velocity"/>
-                <state_interface name="position"/>
-            </joint>
-            <joint name="encoder_right_wheel_joint">
-                <state_interface name="velocity"/>
-                <state_interface name="position"/>
-            </joint> -->
         </ros2_control>
     </xacro:if>
